Commit message: Connect Bob CAD Webots actuators to existing ROS 2 motion commands

File: src/bob_description/urdf/robot.urdf (robot description, URDF)
Before this commit: robot bob, 17 links, 16 joints
Joints:
- removed joint leg0_joint1
- removed joint leg0_joint2
- removed joint leg0_joint3
- removed joint leg1_joint1
- removed joint leg1_joint2
- removed joint leg1_joint3
- removed joint leg2_joint1
- removed joint leg2_joint2
- removed joint leg2_joint3
- removed joint leg3_joint1
- removed joint leg3_joint2
- removed joint leg3_joint3
- added joint joint1_leg0: type revolute, parent leg0_mount, child leg0_joint1_link, origin xyz=-0.137775 -0.086000 0.111950 rpy=0 0 0, axis 0 0 1, limit lower=-1.570796 upper=1.570796 effort=10 velocity=2.618
- added joint joint1_leg1: type revolute, parent leg1_mount, child leg1_joint1_link, origin xyz=-0.139700 0.140000 0.111950 rpy=0 0 0, axis 0 0 1, limit lower=-1.570796 upper=1.570796 effort=10 velocity=2.618
- added joint joint1_leg2: type revolute, parent leg2_mount, child leg2_joint1_link, origin xyz=-0.010300 0.140000 0.111950 rpy=0 0 0, axis 0 0 1, limit lower=-1.570796 upper=1.570796 effort=10 velocity=2.618
- added joint joint1_leg3: type revolute, parent leg3_mount, child leg3_joint1_link, origin xyz=-0.010300 -0.086000 0.111950 rpy=0 0 0, axis 0 0 1, limit lower=-1.570796 upper=1.570796 effort=10 velocity=2.618
- added joint joint3_leg0: type revolute, parent leg0_joint1_link, child leg0_joint2_link, origin xyz=-0.107210 0.025964 -0.010750 rpy=0 0 0, axis 0 1 0, limit lower=-1.570796 upper=1.570796 effort=10 velocity=2.618
- added joint joint3_leg1: type revolute, parent leg1_joint1_link, child leg1_joint2_link, origin xyz=-0.107210 0.025964 -0.010750 rpy=0 0 0, axis 0 1 0, limit lower=-1.570796 upper=1.570796 effort=10 velocity=2.618
- added joint joint3_leg2: type revolute, parent leg2_joint1_link, child leg2_joint2_link, origin xyz=0.107210 -0.025964 -0.010750 rpy=0 0 0, axis 0 1 0, limit lower=-1.570796 upper=1.570796 effort=10 velocity=2.618
- added joint joint3_leg3: type revolute, parent leg3_joint1_link, child leg3_joint2_link, origin xyz=0.107210 -0.025964 -0.010750 rpy=0 0 0, axis 0 1 0, limit lower=-1.570796 upper=1.570796 effort=10 velocity=2.618
- added joint joint4_leg0: type revolute, parent leg0_joint2_link, child leg0_joint3_link, origin xyz=-0.107210 -0.033700 -0.000014 rpy=0 0 0, axis 0 1 0, limit lower=-1.570796 upper=1.570796 effort=10 velocity=2.618
- added joint joint4_leg1: type revolute, parent leg1_joint2_link, child leg1_joint3_link, origin xyz=-0.107210 -0.033700 -0.000014 rpy=0 0 0, axis 0 1 0, limit lower=-1.570796 upper=1.570796 effort=10 velocity=2.618
- added joint joint4_leg2: type revolute, parent leg2_joint2_link, child leg2_joint3_link, origin xyz=0.107210 0.033700 -0.000014 rpy=0 0 0, axis 0 1 0, limit lower=-1.570796 upper=1.570796 effort=10 velocity=2.618
- added joint joint4_leg3: type revolute, parent leg3_joint2_link, child leg3_joint3_link, origin xyz=0.107210 0.033700 -0.000014 rpy=0 0 0, axis 0 1 0, limit lower=-1.570796 upper=1.570796 effort=10 velocity=2.618

File: src/bob_description/urdf/robot.xacro (robot description, xacro)
@@ -7,9 +7,9 @@
     <joint name="${prefix}_mount_fixed" type="fixed"><parent link="base_link"/><child link="${prefix}_mount"/><origin xyz="0 0 0" rpy="0 0 0"/></joint>
     <link name="${prefix}_joint1_link"><visual><origin xyz="${a1}" rpy="0 0 0"/><geometry><mesh filename="package://bob_description/meshes/${prefix}_part1.stl"/></geometry></visual><inertial><mass value="0.2"/><inertia ixx="0.001" iyy="0.001" izz="0.001" ixy="0" ixz="0" iyz="0"/></inertial></link>
-    <joint name="${prefix}_joint1" type="revolute"><parent link="${prefix}_mount"/><child link="${prefix}_joint1_link"/><origin xyz="${a0}" rpy="0 0 0"/><axis xyz="0 0 1"/><limit lower="-1.570796" upper="1.570796" effort="10" velocity="2.618"/></joint>
+    <joint name="joint1_${prefix}" type="revolute"><parent link="${prefix}_mount"/><child link="${prefix}_joint1_link"/><origin xyz="${a0}" rpy="0 0 0"/><axis xyz="0 0 1"/><limit lower="-1.570796" upper="1.570796" effort="10" velocity="2.618"/></joint>
     <link name="${prefix}_joint2_link"><visual><origin xyz="${a2}" rpy="0 0 0"/><geometry><mesh filename="package://bob_description/meshes/${prefix}_part2.stl"/></geometry></visual><inertial><mass value="0.2"/><inertia ixx="0.001" iyy="0.001" izz="0.001" ixy="0" ixz="0" iyz="0"/></inertial></link>
-    <joint name="${prefix}_joint2" type="revolute"><parent link="${prefix}_joint1_link"/><child link="${prefix}_joint2_link"/><origin xyz="${d1}" rpy="0 0 0"/><axis xyz="0 1 0"/><limit lower="-1.570796" upper="1.570796" effort="10" velocity="2.618"/></joint>
+    <joint name="joint3_${prefix}" type="revolute"><parent link="${prefix}_joint1_link"/><child link="${prefix}_joint2_link"/><origin xyz="${d1}" rpy="0 0 0"/><axis xyz="0 1 0"/><limit lower="-1.570796" upper="1.570796" effort="10" velocity="2.618"/></joint>
     <link name="${prefix}_joint3_link"><visual><origin xyz="${a3}" rpy="0 0 0"/><geometry><mesh filename="package://bob_description/meshes/${prefix}_part3.stl"/></geometry></visual><inertial><mass value="0.2"/><inertia ixx="0.001" iyy="0.001" izz="0.001" ixy="0" ixz="0" iyz="0"/></inertial></link>
-    <joint name="${prefix}_joint3" type="revolute"><parent link="${prefix}_joint2_link"/><child link="${prefix}_joint3_link"/><origin xyz="${d2}" rpy="0 0 0"/><axis xyz="0 1 0"/><limit lower="-1.570796" upper="1.570796" effort="10" velocity="2.618"/></joint>
+    <joint name="joint4_${prefix}" type="revolute"><parent link="${prefix}_joint2_link"/><child link="${prefix}_joint3_link"/><origin xyz="${d2}" rpy="0 0 0"/><axis xyz="0 1 0"/><limit lower="-1.570796" upper="1.570796" effort="10" velocity="2.618"/></joint>
   </xacro:macro>
   <xacro:bob_leg prefix="leg0" a0="-0.137775 -0.086000 0.111950" a1="0.137775 0.086000 -0.111950" a2="0.244985 0.060036 -0.101200" a3="0.352195 0.093736 -0.101186" d1="-0.107210 0.025964 -0.010750" d2="-0.107210 -0.033700 -0.000014"/>
