Commit message: HobbyPark 25 kg servos, clean-step walker, Webots fixes and obstacle world
- servo: model the HobbyPark 25 kg coreless servo at 7.4 V (2.45 N m stall,
  ~8 rad/s) from one place (rl/spec.py); CAD pockets/holes (49.5 x 10 mm),
  servo mass, URDF limits and Webots motors all follow it
- walker (rocky_walk.npz = walk_hp4 42M): trained for the new servo with a
  4.5 cm target step height, even steps across legs, bounce penalty,
  stricter pivot rewards (anchor, linear offset, slide, no planted pivot
  leg) and a run-progress reward; ~4 cm even steps, near-zero bounces,
  14 footfalls/rad, faster walk/run; previous walker kept as
  rocky_walk_pivot_mg995.npz
- camera: detection range now derived from marker size and resolution
  (15 cm marker at 1280x720 -> ~5.9 m); Pi node matches
- Webots: add servo rotor inertia to the leg links (fixes knee chatter:
  wobble 2.0 -> 0.3-0.5 rad/s, walk 0.086 -> 0.198 m/s); bridge publishes
  and enables the camera, prints the real servo name; world gets walls,
  tall boxes, steps and rocks, plus an empty rocky_bob_open.wbt
- training: --lr/--target-kl for gentle fine-tunes (avoids collapses),
  terrain blocks up to 7 cm; speed_eval.py, step_eval.py, wobble in
  webots_eval.py
- ignore __pycache__ and Webots .wbproj caches

Co-Authored-By: Claude Opus 5.5 <noreply@anthropic.com>

File: cad/rocky_bob/sim/rocky_bob.urdf (robot description, URDF)
Before this commit: robot rocky_bob, 21 links, 20 joints
Links:
- link leg0_joint1_link: mass 0.1277 -> 0.1366
- link leg0_joint2_link: mass 0.1380 -> 0.1454
- link leg0_joint3_link: mass 0.0726 -> 0.0729
- link leg0_mount: mass 0.0737 -> 0.0812
- link leg1_joint1_link: mass 0.1277 -> 0.1366
- link leg1_joint2_link: mass 0.1380 -> 0.1454
- link leg1_joint3_link: mass 0.0726 -> 0.0729
- link leg1_mount: mass 0.0737 -> 0.0812
- link leg2_joint1_link: mass 0.1277 -> 0.1366
- link leg2_joint2_link: mass 0.1380 -> 0.1454
- link leg2_joint3_link: mass 0.0726 -> 0.0729
- link leg2_mount: mass 0.0737 -> 0.0812
- link leg3_joint1_link: mass 0.1277 -> 0.1366
- link leg3_joint2_link: mass 0.1380 -> 0.1454
- link leg3_joint3_link: mass 0.0726 -> 0.0729
- link leg3_mount: mass 0.0737 -> 0.0812
Joints:
- joint joint1_leg0: limit lower=-1.5708 upper=1.5708 effort=0.94 velocity=5.2 -> lower=-1.5708 upper=1.5708 effort=2.45 velocity=8.0
- joint joint1_leg1: limit lower=-1.5708 upper=1.5708 effort=0.94 velocity=5.2 -> lower=-1.5708 upper=1.5708 effort=2.45 velocity=8.0
- joint joint1_leg2: limit lower=-1.5708 upper=1.5708 effort=0.94 velocity=5.2 -> lower=-1.5708 upper=1.5708 effort=2.45 velocity=8.0
- joint joint1_leg3: limit lower=-1.5708 upper=1.5708 effort=0.94 velocity=5.2 -> lower=-1.5708 upper=1.5708 effort=2.45 velocity=8.0
- joint joint3_leg0: limit lower=-1.5708 upper=1.5708 effort=0.94 velocity=5.2 -> lower=-1.5708 upper=1.5708 effort=2.45 velocity=8.0
- joint joint3_leg1: limit lower=-1.5708 upper=1.5708 effort=0.94 velocity=5.2 -> lower=-1.5708 upper=1.5708 effort=2.45 velocity=8.0
- joint joint3_leg2: limit lower=-1.5708 upper=1.5708 effort=0.94 velocity=5.2 -> lower=-1.5708 upper=1.5708 effort=2.45 velocity=8.0
- joint joint3_leg3: limit lower=-1.5708 upper=1.5708 effort=0.94 velocity=5.2 -> lower=-1.5708 upper=1.5708 effort=2.45 velocity=8.0
- joint joint4_leg0: limit lower=-1.5708 upper=1.5708 effort=0.94 velocity=5.2 -> lower=-1.5708 upper=1.5708 effort=2.45 velocity=8.0
- joint joint4_leg1: limit lower=-1.5708 upper=1.5708 effort=0.94 velocity=5.2 -> lower=-1.5708 upper=1.5708 effort=2.45 velocity=8.0
- joint joint4_leg2: limit lower=-1.5708 upper=1.5708 effort=0.94 velocity=5.2 -> lower=-1.5708 upper=1.5708 effort=2.45 velocity=8.0
- joint joint4_leg3: limit lower=-1.5708 upper=1.5708 effort=0.94 velocity=5.2 -> lower=-1.5708 upper=1.5708 effort=2.45 velocity=8.0
- joint leg0_foot_fixed: origin xyz=0.16000 -0.00150 0 -> xyz=0.16000 -0.00175 0
- joint leg0_mount_fixed: origin xyz=-0.10653 -0.10653 0.06000 rpy=0 0 3.926991 -> xyz=-0.10624 -0.10624 0.06000 rpy=0 0 3.926991
- joint leg1_foot_fixed: origin xyz=0.16000 -0.00150 0 -> xyz=0.16000 -0.00175 0
- joint leg1_mount_fixed: origin xyz=-0.10653 0.10653 0.06000 rpy=0 0 2.356194 -> xyz=-0.10624 0.10624 0.06000 rpy=0 0 2.356194
- joint leg2_foot_fixed: origin xyz=0.16000 -0.00150 0 -> xyz=0.16000 -0.00175 0
- joint leg2_mount_fixed: origin xyz=0.10653 0.10653 0.06000 rpy=0 0 0.785398 -> xyz=0.10624 0.10624 0.06000 rpy=0 0 0.785398
- joint leg3_foot_fixed: origin xyz=0.16000 -0.00150 0 -> xyz=0.16000 -0.00175 0
- joint leg3_mount_fixed: origin xyz=0.10653 -0.10653 0.06000 rpy=0 0 -0.785398 -> xyz=0.10624 -0.10624 0.06000 rpy=0 0 -0.785398

Commit message: Rocky-Bob: lidar, floor sensor, navigation, stairs, self-righting, demos
- Lidar (RPLIDAR C1) on the lid and a ToF floor sensor (VL53L5CX) in the
  nose: CAD mounts, MuJoCo rays, Webots devices, /scan and /tof topics,
  and a live point-cloud viewer (rl/scan_viewer.py)
- Planner navigator: target memory, free-path steering, lidar safety
  layer, stuck escape, and floor-sensor step/cliff detection
- Walker: full servo range, floor heights as inputs, varied stairs
  curriculum (pyramids, flights, kerbs, pits, uneven), stair-quality
  rewards, mixed-difficulty terrain
- Self-righting: learned roll-over plus scripted tidy-up, joint speed
  cap, lidar-contact and impact penalties
- Training loop on demand (scripts/train_more.sh) with best-snapshot
  selection (keep_best.py), and Webots demos (scripts/demo.sh)
- Mustache

Co-Authored-By: Claude Opus 5.5 <noreply@anthropic.com>

File: cad/rocky_bob/sim/rocky_bob.urdf (robot description, URDF)
Before this commit: robot rocky_bob, 21 links, 20 joints
Links:
- link base_link: mass 0.6718 -> 0.7748; geometry collision box size=0.05560 0.05560 0.04130; collision box size=0.06400 0.06400 0.02600
